Commit message: ridgeback_dual_ur done

File: urdf/gazebo/mbot/mbot_ur_test.xacro (robot description, xacro)
@@ -1,5 +1,5 @@
 <?xml version="1.0"?>
 <robot name="mbot" xmlns:xacro="http://ros.org/wiki/xacro">
-    <!--xacro:include filename="$(find ridgeback_description_mbot)/urdf/gazebo/mbot/ridgeback_dual_ur5_description.urdf.xacro" /-->
-    <xacro:include filename="$(find ridgeback_ur_description)/urdf/ridgeback_dual_ur5_description.urdf.xacro" />
+    <xacro:include filename="$(find ridgeback_description_mbot)/urdf/gazebo/mbot/ridgeback_dual_ur5_description.urdf.xacro" />
+    <!--xacro:include filename="$(find ridgeback_description_mbot)/urdf/ridgeback_dual_ur5_description.urdf.xacro" /-->
 </robot>

File: urdf/gazebo/mbot/ridgeback_dual_ur5_description.urdf.xacro (robot description, xacro)
@@ -11,5 +11,5 @@
     <origin xyz="$(optenv RIDGEBACK_RIGHT_UR_XYZ 0.21 -0.20 0.0)" rpy="$(optenv RIDGEBACK_RIGHT_UR_RPY 0 0 0)"/>
   </joint>
-  <xacro:include filename="$(find ur_description)/urdf/ur5.urdf.xacro" />
+  <xacro:include filename="$(find ridgeback_description_mbot)/urdf/ur5/ur5.urdf.xacro" />
   <!-- common stuff -->
   <xacro:include filename="$(find ridgeback_description_mbot)/urdf/ur5/common.gazebo.xacro" />

File: urdf/ur5/ur.transmission.xacro (robot description, xacro)
@@ -5,5 +5,5 @@
       <type>transmission_interface/SimpleTransmission</type>
       <joint name="${prefix}shoulder_pan_joint">
-        <hardwareInterface>hardware_interface/PositionJointInterface</hardwareInterface>
+        <hardwareInterface>hardware_interface/EffortJointInterface</hardwareInterface>
       </joint>
       <actuator name="${prefix}shoulder_pan_motor">
@@ -14,5 +14,5 @@
       <type>transmission_interface/SimpleTransmission</type>
       <joint name="${prefix}shoulder_lift_joint">
-        <hardwareInterface>hardware_interface/PositionJointInterface</hardwareInterface>
+        <hardwareInterface>hardware_interface/EffortJointInterface</hardwareInterface>
       </joint>
       <actuator name="${prefix}shoulder_lift_motor">
@@ -23,5 +23,5 @@
       <type>transmission_interface/SimpleTransmission</type>
       <joint name="${prefix}elbow_joint">
-        <hardwareInterface>hardware_interface/PositionJointInterface</hardwareInterface>
+        <hardwareInterface>hardware_interface/EffortJointInterface</hardwareInterface>
       </joint>
       <actuator name="${prefix}elbow_motor">
@@ -32,5 +32,5 @@
       <type>transmission_interface/SimpleTransmission</type>
       <joint name="${prefix}wrist_1_joint">
-        <hardwareInterface>hardware_interface/PositionJointInterface</hardwareInterface>
+        <hardwareInterface>hardware_interface/EffortJointInterface</hardwareInterface>
       </joint>
       <actuator name="${prefix}wrist_1_motor">
@@ -41,5 +41,5 @@
       <type>transmission_interface/SimpleTransmission</type>
       <joint name="${prefix}wrist_2_joint">
-        <hardwareInterface>hardware_interface/PositionJointInterface</hardwareInterface>
+        <hardwareInterface>hardware_interface/EffortJointInterface</hardwareInterface>
       </joint>
       <actuator name="${prefix}wrist_2_motor">
@@ -50,5 +50,5 @@
       <type>transmission_interface/SimpleTransmission</type>
       <joint name="${prefix}wrist_3_joint">
-        <hardwareInterface>hardware_interface/PositionJointInterface</hardwareInterface>
+        <hardwareInterface>hardware_interface/EffortJointInterface</hardwareInterface>
       </joint>
       <actuator name="${prefix}wrist_3_motor">

File: urdf/ur5/ur5.urdf.xacro (robot description, xacro)
@@ -126,5 +126,5 @@
       <parent link="${prefix}shoulder_link" />
       <child link = "${prefix}upper_arm_link" />
-      <origin xyz="0.0 ${shoulder_offset} 0.0" rpy="0.0 ${pi / 2.0} 0.0" />
+      <origin xyz="0.0 ${shoulder_offset} 0.0" rpy="0.0 ${pi / 2.0-pi / 2.0} 0.0" />
       <axis xyz="0 1 0" />
       <xacro:unless value="${joint_limited}">
