Commit message: ridgeback_dualur_allegro_hand done

File: urdf/allergo_hand/dual_allegro_hand.xacro (robot description, xacro)
@@ -1,16 +1,15 @@
 <?xml version="1.0"?>
 <robot name="ur_allegro_ridgeback" xmlns:xacro="http://ros.org/wiki/xacro">
-    <xacro:include filename="$(find allegro_hand_description)/allegro_hand_description_right_tra.urdf" />
-    <xacro:include filename="$(find allegro_hand_description)/allegro_hand_description_left_tra.urdf" />
-<ridgeback/>
+    <xacro:include filename="$(find allegro_hand_description)/allegro_hand_description_right.urdf" />
+    <!--xacro:include filename="$(find allegro_hand_description)/allegro_hand_description_left_tra.urdf" /-->
     <joint name="connect_joint" type="fixed">
-	<origin xyz="0 0 0.095" rpy="0 0 0"/>
-	<parent link="right_ur_arm_tool0"/>
-	<child link="palm_link"/>
+	    <origin xyz="0 0 0.095" rpy="0 0 0"/>
+	    <parent link="right_ur_arm_tool0"/>
+	    <child link="palm_link"/>
     </joint>
-    <joint name="connect_joint1" type="fixed">
-	<origin xyz="0 0 0.095" rpy="0 0 0"/>
-	<parent link="left_ur_arm_tool0"/>
-	<child link="left_palm_link"/>
-    </joint>
+    <!--joint name="connect_joint1" type="fixed">
+	    <origin xyz="0 0 0.095" rpy="0 0 0"/>
+	    <parent link="left_ur_arm_tool0"/>
+	    <child link="left_palm_link"/>
+    </joint-->
 </robot>

File: urdf/gazebo/mbot/mbot_ur_test.xacro (robot description, xacro)
@@ -2,4 +2,4 @@
 <robot name="mbot" xmlns:xacro="http://ros.org/wiki/xacro">
     <xacro:include filename="$(find ridgeback_description_mbot)/urdf/gazebo/mbot/ridgeback_dual_ur5_description.urdf.xacro" />
-    <!--xacro:include filename="$(find ridgeback_description_mbot)/urdf/allergo_hand/dual_allegro_hand.xacro" /-->
+    <xacro:include filename="$(find ridgeback_description_mbot)/urdf/allergo_hand/dual_allegro_hand.xacro" />
 </robot>
